File: KiCad_Files/MPU6050_Sensor/MPU6050_I2c/MPU6050_I2c.kicad_pcb (KiCad board)
At the start: 4 copper layers, 40 x 40 mm, 11 parts, among them J1 Conn_01x05, SW1 SW_SPDT, U1 MPU-6050

Commit message: Working Version of MPU6050 Library
Parts:
- added REF**: Symbol_GNU-Logo_SilkscreenTop, Symbol:Symbol_GNU-Logo_SilkscreenTop, F.Cu at (127.4, 72.6)
- added REF**: KiCad-Logo2_5mm_SilkScreen, Symbol:KiCad-Logo2_5mm_SilkScreen, F.Cu at (156.0, 79.0)
Other:
- board text added: "JLCJLCJLCJLC"
