File: PCB/TB6612_MotorBridge/TB6612_MotorBridge/TB6612_MotorBridge.kicad_sch (KiCad schematic)
At the start: 14 parts, among them J1 Screw_Terminal_01x02, J4 Conn_01x02, J5 Conn_01x02, J8 Conn_01x05, J9 Conn_01x05, U1 TB6612FNG, U2 DMG3415U-7

Commit message: Updated PCB Main and MotorBridge with Pins for Encoder
Parts:
- removed J4, J5: Conn_01x02, Connector_JST:JST_XH_B2B-XH-A_1x02_P2.50mm_Vertical, symbol Connector_Generic:Conn_01x02
- removed J8, J9: Conn_01x05, Connector_JST:JST_XH_B5B-XH-AM_1x05_P2.50mm_Vertical, symbol Connector_Generic:Conn_01x05
- added J4, J5: Conn_01x06, Connector_JST:JST_XH_B6B-XH-A_1x06_P2.50mm_Vertical, symbol Connector_Generic:Conn_01x06
- added J8, J9: Conn_01x07, Connector_JST:JST_XH_B7B-XH-A_1x07_P2.50mm_Vertical, symbol Connector_Generic:Conn_01x07
Connections:
- net +3.3V: now also J4.5 (Pin_5), J5.5 (Pin_5), J8.1 (Pin_1), J9.1 (Pin_1)
- net A1: now also J8.3 (Pin_3)
- net A2: now also J8.4 (Pin_4)
- net B1: now also J9.3 (Pin_3)
- net B2: now also J9.4 (Pin_4)
- net GND: now also J4.2 (Pin_2), J5.2 (Pin_2), J8.7 (Pin_7), J9.7 (Pin_7)
- net MA1: now also J4.1 (Pin_1)
- net MA2: now also J4.6 (Pin_6)
- net MB1: now also J5.1 (Pin_1)
- net MB2: now also J5.6 (Pin_6)
- net PWM_A: now also J8.2 (Pin_2)
- net PWM_B: now also J9.2 (Pin_2)
- new net EA1: J4.3 (Pin_3), J8.5 (Pin_5)
- new net EA2: J4.4 (Pin_4), J8.6 (Pin_6)
- new net EB1: J5.3 (Pin_3), J9.5 (Pin_5)
- new net EB2: J5.4 (Pin_4), J9.6 (Pin_6)
