File: PCB/MPU6050_Sensor/MPU6050_I2c.kicad_pcb (KiCad board)
At the start: 4 copper layers, 40 x 40 mm, 13 parts, among them J1 Conn_01x05, SW1 SW_SPDT, U1 MPU-6050

Commit message: Converted all vias to through-hole
Changed lines of the file:
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@@
   (segment (start 140.3 83.190685) (end 139.990685 83.5) (width 0.25) (layer "F.Cu") (net 4))
   (segment (start 139.990685 83.5) (end 138 83.5) (width 0.25) (layer "F.Cu") (net 4))
+  (via (at 136.5 69.5) (size 0.8) (drill 0.4) (layers "F.Cu" "B.Cu") (net 4))
+  (via (at 130.75 85.5) (size 0.8) (drill 0.4) (layers "F.Cu" "B.Cu") (net 4))
+  (via (at 133 83.25) (size 0.8) (drill 0.4) (layers "F.Cu" "B.Cu") (net 4))
+  (via (at 136.5 68.75) (size 0.8) (drill 0.4) (layers "F.Cu" "B.Cu") (net 4))
   (via (at 144.5 79.75) (size 0.8) (drill 0.4) (layers "F.Cu" "B.Cu") (net 4))
   (via (at 138 83.5) (size 0.8) (drill 0.4) (layers "F.Cu" "B.Cu") (net 4))
@@
   (segment (start 131.25 74.75) (end 131.25 81.5) (width 1) (layer "In2.Cu") (net 4))
   (segment (start 144.5 79.5) (end 144.5 79.75) (width 1) (layer "In2.Cu") (net 4))
-  (via blind (at 136.5 69.5) (size 0.8) (drill 0.4) (layers "In2.Cu" "B.Cu") (net 4))
-  (via blind (at 130.75 85.5) (size 0.8) (drill 0.4) (layers "In2.Cu" "B.Cu") (net 4))
-  (via blind (at 133 83.25) (size 0.8) (drill 0.4) (layers "In2.Cu" "B.Cu") (net 4))
-  (via blind (at 136.5 68.75) (size 0.8) (drill 0.4) (layers "In2.Cu" "B.Cu") (net 4))
   (segment (start 136.5 68.75) (end 136.5 69.5) (width 1) (layer "B.Cu") (net 4))
   (segment (start 136.5 67) (end 136.5 68.75) (width 1) (layer "B.Cu") (net 4))
