File: PCB/VL53L0X_Sensor/VL53L0X_I2c.kicad_pcb (KiCad board)
At the start: 4 copper layers, 50 x 20 mm, 11 parts, among them J1 Conn_01x05, U1 VL53L1CXV0FY1

Commit message: Converted all vias to through-hole
Changed lines of the file:
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@@
       (stroke (width 0.1) (type solid)) (layer "F.Fab"))
     (pad "" np_thru_hole circle (at -1.6 2 180) (size 1.2 1.2) (drill 1.2) (layers "*.Cu" "*.Mask"))
-    (pad "1" thru_hole roundrect (at 0 0 180) (size 1.7 1.95) (drill 0.95) (layers "*.Cu" "*.Mask") (roundrect_rratio 0.147059)
+    (pad "1" thru_hole roundrect (at 0 0 180) (size 1.7 1.95) (drill 0.95) (layers "*.Cu" "*.Mask") (roundrect_rratio 0.1470588235)
       (net 1 "+3.3V") (pinfunction "Pin_1") (pintype "passive"))
     (pad "2" thru_hole oval (at 2.5 0 180) (size 1.7 1.95) (drill 0.95) (layers "*.Cu" "*.Mask")
@@
   (segment (start 122 69.4) (end 122.25 69.15) (width 0.5) (layer "F.Cu") (net 1))
   (segment (start 122 71) (end 122 69.4) (width 0.5) (layer "F.Cu") (net 1))
+  (via (at 131 68) (size 0.8) (drill 0.4) (layers "F.Cu" "B.Cu") (net 1))
   (via (at 120 68) (size 0.8) (drill 0.4) (layers "F.Cu" "B.Cu") (net 1))
-  (via blind (at 122 71) (size 0.8) (drill 0.4) (layers "F.Cu" "In2.Cu") (net 1))
+  (via (at 128.939668 74.879337) (size 0.8) (drill 0.4) (layers "F.Cu" "B.Cu") (net 1))
+  (via (at 122 71) (size 0.8) (drill 0.4) (layers "F.Cu" "B.Cu") (net 1))
+  (via (at 120 69) (size 0.8) (drill 0.4) (layers "F.Cu" "B.Cu") (net 1))
   (segment (start 127.060331 73) (end 124 73) (width 1) (layer "In2.Cu") (net 1))
   (segment (start 128.939668 74.879337) (end 129.120663 74.879337) (width 0.25) (layer "In2.Cu") (net 1))
@@
   (segment (start 128.939668 74.879337) (end 127.060331 73) (width 1) (layer "In2.Cu") (net 1))
   (segment (start 131 73) (end 131 68) (width 1) (layer "In2.Cu") (net 1))
-  (via blind (at 131 68) (size 0.8) (drill 0.4) (layers "In2.Cu" "B.Cu") (net 1))
-  (via blind (at 128.939668 74.879337) (size 0.8) (drill 0.4) (layers "In2.Cu" "B.Cu") (net 1))
-  (via blind (at 120 69) (size 0.8) (drill 0.4) (layers "In2.Cu" "B.Cu") (net 1))
   (segment (start 135.08 77) (end 136 76.08) (width 1) (layer "B.Cu") (net 1))
   (segment (start 120 68) (end 120 67.5) (width 1) (layer "B.Cu") (net 1))
